Commit message: Kinematics added(thumb rotation not working)

File: Data/robot.urdf (robot description, URDF)
Before this commit: robot onshape, 21 links, 20 joints
Links:
- removed link fingertip_2_tip
- removed link fingertip_3_tip
- removed link fingertip_tip
- removed link thumb_tip
Joints:
- removed joint fingertip_2_tip_joint
- removed joint fingertip_3_tip_joint
- removed joint fingertip_tip_joint
- removed joint thumb_tip_joint
