Commit message: Sim2Real based Proprioceptive Recognition

File: Data/Leap_Model/mujoco_robot.urdf (robot description, URDF)
Before this commit: robot onshape, 17 links, 16 joints
Joints:
- joint 0: limit lower=-1.047 upper=1.047 effort=0.95 velocity=8.48 -> lower=-1.3089969389957472 upper=1.047 effort=0.95 velocity=8.48
- joint 13: limit lower=-0.47 upper=2.443 effort=0.95 velocity=8.48 -> lower=-0.47 upper=3.141592653589793 effort=0.95 velocity=8.48
- joint 14: limit lower=-1.20 upper=1.90 effort=0.95 velocity=8.48 -> lower=-1.20 upper=1.9198621771937625 effort=0.95 velocity=8.48
- joint 8: limit lower=-1.047 upper=1.047 effort=0.95 velocity=8.48 -> lower=-1.047 upper=1.3089969389957472 effort=0.95 velocity=8.48

File: Data/Leap_Model/robot.urdf (robot description, URDF)
Before this commit: robot onshape, 17 links, 16 joints
Joints:
- joint 0: limit lower=-1.047 upper=1.047 effort=0.95 velocity=8.48 -> lower=-1.3089969389957472 upper=1.047 effort=0.95 velocity=8.48
- joint 13: limit lower=-0.47 upper=2.443 effort=0.95 velocity=8.48 -> lower=-0.47 upper=3.141592653589793 effort=0.95 velocity=8.48
- joint 14: limit lower=-1.20 upper=1.90 effort=0.95 velocity=8.48 -> lower=-1.20 upper=1.9198621771937625 effort=0.95 velocity=8.48
- joint 8: limit lower=-1.047 upper=1.047 effort=0.95 velocity=8.48 -> lower=-1.047 upper=1.3089969389957472 effort=0.95 velocity=8.48
